File: EasyCheck_rev2/EasyCheck_rev2_interface.brd (EAGLE design)
At the start: 170 x 40 mm, 18 parts

Commit message: Corrected hardware files
Connections:
- net /SS: now also JP1.7; no longer JP1.9
- net MOSI: now also JP1.9; no longer JP1.5
- net SCK: now also JP1.5; no longer JP1.7
Routing:
- net SCK: track 15.0 -> 22.6 mm
- net /SS: track 17.0 -> 12.6 mm
- net MISO: track 17.1 -> 13.7 mm
- net MOSI: track 15.1 -> 12.1 mm
- net LCD_DC: track 14.4 -> 12.6 mm
Changed lines of the file:
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@@
 <wire x1="5.285" y1="6.415" x2="5.18" y2="6.31" width="0.254" layer="1"/>
 <wire x1="5.18" y1="6.31" x2="2.7" y2="6.31" width="0.254" layer="1"/>
-<wire x1="-86.335" y1="-5.28" x2="-87.515" y2="-4.1" width="0.254" layer="1"/>
-<wire x1="-87.515" y1="-4.1" x2="-87.55" y2="-4.1" width="0.254" layer="1"/>
-<wire x1="-87.55" y1="-4.1" x2="-87.55" y2="5.3" width="0.254" layer="1"/>
-<wire x1="-87.55" y1="5.3" x2="-81.5636" y2="11.2864" width="0.254" layer="1"/>
+<wire x1="-81.5636" y1="11.2864" x2="-87.55" y2="5.3" width="0.254" layer="1"/>
 <wire x1="-69.8864" y1="11.2864" x2="-60.8564" y2="2.2564" width="0.254" layer="1"/>
 <wire x1="-1.3536" y1="2.2564" x2="2.7" y2="6.31" width="0.254" layer="1"/>
 <wire x1="-81.5636" y1="11.2864" x2="-69.8864" y2="11.2864" width="0.254" layer="1"/>
 <wire x1="-60.8564" y1="2.2564" x2="-1.3536" y2="2.2564" width="0.254" layer="1"/>
+<wire x1="-87.55" y1="5.3" x2="-87.55" y2="-4.065" width="0.254" layer="1"/>
+<wire x1="-87.55" y1="-4.065" x2="-86.335" y2="-5.28" width="0.254" layer="1"/>
 </signal>
 <signal name="N$2">
@@
 </signal>
 <signal name="MOSI">
-<contactref element="JP1" pad="5"/>
 <contactref element="JP2" pad="4"/>
-<wire x1="-78.75" y1="-9.53" x2="-79.95" y2="-9.53" width="0.254" layer="16"/>
-<wire x1="-79.95" y1="-9.53" x2="-85.28" y2="-4.2" width="0.254" layer="16"/>
-<wire x1="-85.28" y1="-4.2" x2="-86.725" y2="-4.2" width="0.254" layer="16"/>
-<wire x1="-88.875" y1="-0.2" x2="-87.725" y2="-1.35" width="0.254" layer="16"/>
-<wire x1="-87.725" y1="-1.35" x2="-87.725" y2="-3.2" width="0.254" layer="16"/>
-<wire x1="-86.725" y1="-4.2" x2="-87.725" y2="-3.2" width="0.254" layer="16"/>
+<contactref element="JP1" pad="9"/>
+<wire x1="-78.75" y1="-9.53" x2="-82.82" y2="-9.53" width="0.254" layer="1"/>
+<wire x1="-85.85" y1="-6.5" x2="-88" y2="-6.5" width="0.254" layer="1"/>
+<wire x1="-88" y1="-6.5" x2="-88.875" y2="-5.625" width="0.254" layer="1"/>
+<wire x1="-88.875" y1="-5.625" x2="-88.875" y2="-5.28" width="0.254" layer="1"/>
+<wire x1="-82.82" y1="-9.53" x2="-85.85" y2="-6.5" width="0.254" layer="1"/>
 </signal>
 <signal name="SCK">
-<contactref element="JP1" pad="7"/>
 <contactref element="JP2" pad="3"/>
 <wire x1="-80.045" y1="-12.07" x2="-78.75" y2="-12.07" width="0.254" layer="16"/>
-<wire x1="-86.575" y1="-6.69" x2="-87.775" y2="-5.49" width="0.254" layer="16"/>
-<wire x1="-88.875" y1="-2.74" x2="-87.775" y2="-3.84" width="0.254" layer="16"/>
-<wire x1="-87.775" y1="-3.84" x2="-87.775" y2="-5.49" width="0.254" layer="16"/>
-<wire x1="-85.425" y1="-6.69" x2="-86.575" y2="-6.69" width="0.254" layer="16"/>
-<wire x1="-80.045" y1="-12.07" x2="-85.425" y2="-6.69" width="0.254" layer="16"/>
+<contactref element="JP1" pad="5"/>
+<wire x1="-78.75" y1="-12.07" x2="-82.98" y2="-12.07" width="0.254" layer="1"/>
+<wire x1="-89.3063625" y1="-8.8614" x2="-89.9164" y2="-8.2513625" width="0.254" layer="1"/>
+<wire x1="-89.9164" y1="-8.2513625" x2="-89.9164" y2="-8.2336" width="0.254" layer="1"/>
+<wire x1="-89.9164" y1="-8.2336" x2="-90.05" y2="-8.1" width="0.254" layer="1"/>
+<wire x1="-86.1886" y1="-8.8614" x2="-89.3063625" y2="-8.8614" width="0.254" layer="1"/>
+<wire x1="-90.05" y1="-8.1" x2="-90.05" y2="-1.375" width="0.254" layer="1"/>
+<wire x1="-90.05" y1="-1.375" x2="-88.875" y2="-0.2" width="0.254" layer="1"/>
+<wire x1="-82.98" y1="-12.07" x2="-86.1886" y2="-8.8614" width="0.254" layer="1"/>
 </signal>
 <signal name="MISO">
+<contactref element="JP2" pad="8"/>
 <contactref element="JP1" pad="11"/>
-<contactref element="JP2" pad="8"/>
-<wire x1="-88.875" y1="-7.82" x2="-87.745" y2="-8.95" width="0.254" layer="1"/>
-<wire x1="-81.4" y1="-4.6" x2="-81.4" y2="-0.27" width="0.254" layer="1"/>
-<wire x1="-81.4" y1="-0.27" x2="-80.5" y2="0.63" width="0.254" layer="1"/>
-<wire x1="-87.745" y1="-8.95" x2="-85.75" y2="-8.95" width="0.254" layer="1"/>
-<wire x1="-85.75" y1="-8.95" x2="-81.4" y2="-4.6" width="0.254" layer="1"/>
-<wire x1="-80.5" y1="0.63" x2="-78.75" y2="0.63" width="0.254" layer="1"/>
+<wire x1="-88.875" y1="-7.82" x2="-87.555" y2="-6.5" width="0.254" layer="16"/>
+<wire x1="-87.555" y1="-6.5" x2="-85.8247625" y2="-6.5" width="0.254" layer="16"/>
+<wire x1="-78.75" y1="0.5747625" x2="-78.75" y2="0.63" width="0.254" layer="16"/>
+<wire x1="-85.8247625" y1="-6.5" x2="-78.75" y2="0.5747625" width="0.254" layer="16"/>
 </signal>
 <signal name="/SS">
-<contactref element="JP1" pad="9"/>
 <contactref element="JP2" pad="9"/>
-<wire x1="-85.775" y1="-6.63" x2="-87.525" y2="-6.63" width="0.254" layer="1"/>
-<wire x1="-88.875" y1="-5.28" x2="-87.525" y2="-6.63" width="0.254" layer="1"/>
-<wire x1="-85.775" y1="-6.63" x2="-82.5" y2="-3.355" width="0.254" layer="1"/>
-<wire x1="-82.5" y1="-3.355" x2="-82.5" y2="0.45" width="0.254" layer="1"/>
-<wire x1="-82.5" y1="0.45" x2="-79.78" y2="3.17" width="0.254" layer="1"/>
-<wire x1="-79.78" y1="3.17" x2="-78.75" y2="3.17" width="0.254" layer="1"/>
+<contactref element="JP1" pad="7"/>
+<wire x1="-88.875" y1="-2.74" x2="-87.535" y2="-1.4" width="0.254" layer="16"/>
+<wire x1="-83.32" y1="-1.4" x2="-78.75" y2="3.17" width="0.254" layer="16"/>
+<wire x1="-87.535" y1="-1.4" x2="-83.32" y2="-1.4" width="0.254" layer="16"/>
 </signal>
 <signal name="LCD_DC">
 <contactref element="JP2" pad="6"/>
 <contactref element="JP1" pad="13"/>
-<wire x1="-85.8925" y1="-11.5425" x2="-87.325" y2="-11.5425" width="0.254" layer="1"/>
-<wire x1="-88.875" y1="-10.36" x2="-88.975" y2="-10.26" width="0.254" layer="1"/>
-<wire x1="-88.975" y1="-9.8925" x2="-88.975" y2="-10.26" width="0.254" layer="1"/>
-<wire x1="-87.325" y1="-11.5425" x2="-88.975" y2="-9.8925" width="0.254" layer="1"/>
-<wire x1="-78.75" y1="-4.45" x2="-78.8" y2="-4.45" width="0.254" layer="1"/>
-<wire x1="-78.8" y1="-4.45" x2="-85.8925" y2="-11.5425" width="0.254" layer="1"/>
+<wire x1="-88.875" y1="-10.36" x2="-87.615" y2="-9.1" width="0.254" layer="16"/>
+<wire x1="-83.4" y1="-9.1" x2="-78.75" y2="-4.45" width="0.254" layer="16"/>
+<wire x1="-87.615" y1="-9.1" x2="-83.4" y2="-9.1" width="0.254" layer="16"/>
 </signal>
 <signal name="N$1">
@@
 <contactref element="JP2" pad="5"/>
 <contactref element="JP1" pad="16"/>
-<wire x1="-86.335" y1="-12.9" x2="-84.66" y2="-12.9" width="0.254" layer="1"/>
-<wire x1="-84.66" y1="-12.9" x2="-78.75" y2="-6.99" width="0.254" layer="1"/>
+<wire x1="-86.335" y1="-12.9" x2="-84.66" y2="-12.9" width="0.254" layer="16"/>
+<wire x1="-84.66" y1="-12.9" x2="-78.75" y2="-6.99" width="0.254" layer="16"/>
 </signal>
 </signals>
