File: EasyCheck_rev2/EasyCheck_rev2_interface.sch (EAGLE design)
At the start: 18 parts

Commit message: Corrected hardware files
Connections:
- net /SS: now also JP1.7; no longer JP1.9
- net MOSI: now also JP1.9; no longer JP1.5
- net SCK: now also JP1.5; no longer JP1.7
Changed lines of the file:
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@@
 <setting verticaltext="up"/>
 </settings>
-<grid distance="0.1" unitdist="inch" unit="inch" style="lines" multiple="1" display="yes" altdistance="0.01" altunitdist="inch" altunit="inch"/>
+<grid distance="0.1" unitdist="inch" unit="inch" style="lines" multiple="1" display="no" altdistance="0.01" altunitdist="inch" altunit="inch"/>
 <layers>
 <layer number="1" name="Top" color="4" fill="1" visible="no" active="no"/>
@@
 <net name="MOSI" class="0">
 <segment>
+<wire x1="147.32" y1="-101.6" x2="127" y2="-101.6" width="0.1524" layer="91"/>
+<label x="127" y="-101.6" size="1.27" layer="95" font="vector" rot="R180" xref="yes"/>
+<pinref part="JP2" gate="A" pin="4"/>
+</segment>
+<segment>
+<wire x1="121.92" y1="-38.1" x2="114.3" y2="-38.1" width="0.1524" layer="91"/>
+<label x="114.3" y="-38.1" size="1.27" layer="95" font="vector" rot="R180" xref="yes"/>
+<pinref part="JP1" gate="A" pin="9"/>
+</segment>
+</net>
+<net name="SCK" class="0">
+<segment>
+<wire x1="147.32" y1="-99.06" x2="127" y2="-99.06" width="0.1524" layer="91"/>
+<label x="127" y="-99.06" size="1.27" layer="95" font="vector" rot="R180" xref="yes"/>
+<pinref part="JP2" gate="A" pin="3"/>
+</segment>
+<segment>
 <wire x1="121.92" y1="-33.02" x2="114.3" y2="-33.02" width="0.1524" layer="91"/>
 <label x="114.3" y="-33.02" size="1.27" layer="95" font="vector" rot="R180" xref="yes"/>
 <pinref part="JP1" gate="A" pin="5"/>
 </segment>
-<segment>
-<wire x1="147.32" y1="-101.6" x2="127" y2="-101.6" width="0.1524" layer="91"/>
-<label x="127" y="-101.6" size="1.27" layer="95" font="vector" rot="R180" xref="yes"/>
-<pinref part="JP2" gate="A" pin="4"/>
-</segment>
-</net>
-<net name="SCK" class="0">
+</net>
+<net name="MISO" class="0">
+<segment>
+<wire x1="147.32" y1="-111.76" x2="127" y2="-111.76" width="0.1524" layer="91"/>
+<label x="127" y="-111.76" size="1.27" layer="95" font="vector" rot="R180" xref="yes"/>
+<pinref part="JP2" gate="A" pin="8"/>
+</segment>
+<segment>
+<wire x1="121.92" y1="-40.64" x2="114.3" y2="-40.64" width="0.1524" layer="91"/>
+<label x="114.3" y="-40.64" size="1.27" layer="95" font="vector" rot="R180" xref="yes"/>
+<pinref part="JP1" gate="A" pin="11"/>
+</segment>
+</net>
+<net name="/SS" class="0">
+<segment>
+<wire x1="147.32" y1="-114.3" x2="127" y2="-114.3" width="0.1524" layer="91"/>
+<label x="127" y="-114.3" size="1.27" layer="95" font="vector" rot="R180" xref="yes"/>
+<pinref part="JP2" gate="A" pin="9"/>
+</segment>
 <segment>
 <wire x1="121.92" y1="-35.56" x2="114.3" y2="-35.56" width="0.1524" layer="91"/>
@@
 <pinref part="JP1" gate="A" pin="7"/>
 </segment>
-<segment>
-<wire x1="147.32" y1="-99.06" x2="127" y2="-99.06" width="0.1524" layer="91"/>
-<label x="127" y="-99.06" size="1.27" layer="95" font="vector" rot="R180" xref="yes"/>
-<pinref part="JP2" gate="A" pin="3"/>
-</segment>
-</net>
-<net name="MISO" class="0">
-<segment>
-<wire x1="121.92" y1="-40.64" x2="114.3" y2="-40.64" width="0.1524" layer="91"/>
-<label x="114.3" y="-40.64" size="1.27" layer="95" font="vector" rot="R180" xref="yes"/>
-<pinref part="JP1" gate="A" pin="11"/>
-</segment>
-<segment>
-<wire x1="147.32" y1="-111.76" x2="127" y2="-111.76" width="0.1524" layer="91"/>
-<label x="127" y="-111.76" size="1.27" layer="95" font="vector" rot="R180" xref="yes"/>
-<pinref part="JP2" gate="A" pin="8"/>
-</segment>
-</net>
-<net name="/SS" class="0">
-<segment>
-<wire x1="121.92" y1="-38.1" x2="114.3" y2="-38.1" width="0.1524" layer="91"/>
-<label x="114.3" y="-38.1" size="1.27" layer="95" font="vector" rot="R180" xref="yes"/>
-<pinref part="JP1" gate="A" pin="9"/>
-</segment>
-<segment>
-<wire x1="147.32" y1="-114.3" x2="127" y2="-114.3" width="0.1524" layer="91"/>
-<label x="127" y="-114.3" size="1.27" layer="95" font="vector" rot="R180" xref="yes"/>
-<pinref part="JP2" gate="A" pin="9"/>
-</segment>
-</net>
+</net>
