File: EasyCheck_rev2/Easycheck_rev2_motherboard.sch (EAGLE design)
At the start: 61 parts, among them J1 DC-044-20A, J2 CORTEX_DEBUG_PTH, Q1 DMG3415U, Q2 SI7465DP, T1 DS18B20, T2 MMBT2222A, U1 LM5085, U2 AP2114H-3.3V- 1A, U3 ATSAMD21G18A-AU, X1 JST-XH-02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

Commit message: Corrected hardware files
Connections:
- net /SS: now also JP2.7, U3.PA18/I2/SERCOM1+3.2; no longer JP2.9, U3.PA19/I3/SERCOM1+3.3/I2SD0
- net FAN0: now also U3.PA06/EINT6/AIN6/SERCOM0.2; no longer U3.PB09/I9/AIN3/SERCOM4.1
- net FAN0_SPEED: now also U3.PB09/I9/AIN3/SERCOM4.1; no longer U3.PA06/EINT6/AIN6/SERCOM0.2
- net MOSI: now also JP2.9, U3.PA19/I3/SERCOM1+3.3/I2SD0; no longer JP2.5, U3.PA17/I2C/I1/SERCOM1+3.1
- net SCK: now also JP2.5, U3.PA17/I2C/I1/SERCOM1+3.1; no longer JP2.7, U3.PA18/I2/SERCOM1+3.2
Changed lines of the file:
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@@
 <setting verticaltext="up"/>
 </settings>
-<grid distance="0.1" unitdist="inch" unit="inch" style="lines" multiple="1" display="yes" altdistance="0.01" altunitdist="inch" altunit="inch"/>
+<grid distance="0.1" unitdist="inch" unit="inch" style="lines" multiple="1" display="no" altdistance="0.01" altunitdist="inch" altunit="inch"/>
 <layers>
 <layer number="1" name="Top" color="4" fill="1" visible="no" active="no"/>
@@
 </segment>
 </net>
-<net name="MOSI" class="0">
+<net name="SCK" class="0">
+<segment>
+<wire x1="218.44" y1="-223.52" x2="210.82" y2="-223.52" width="0.1524" layer="91"/>
+<label x="210.82" y="-223.52" size="1.27" layer="95" font="vector" rot="R180" xref="yes"/>
+<pinref part="JP2" gate="A" pin="5"/>
+</segment>
 <segment>
 <wire x1="320.04" y1="-78.74" x2="309.88" y2="-78.74" width="0.1524" layer="91"/>
 <label x="309.88" y="-78.74" size="1.27" layer="95" font="vector" rot="R180" xref="yes"/>
 <pinref part="U3" gate="G$1" pin="PA17/I2C/I1/SERCOM1+3.1"/>
-</segment>
-<segment>
-<wire x1="218.44" y1="-223.52" x2="210.82" y2="-223.52" width="0.1524" layer="91"/>
-<label x="210.82" y="-223.52" size="1.27" layer="95" font="vector" rot="R180" xref="yes"/>
-<pinref part="JP2" gate="A" pin="5"/>
-</segment>
-</net>
-<net name="SCK" class="0">
-<segment>
-<wire x1="320.04" y1="-81.28" x2="309.88" y2="-81.28" width="0.1524" layer="91"/>
-<label x="309.88" y="-81.28" size="1.27" layer="95" font="vector" rot="R180" xref="yes"/>
-<pinref part="U3" gate="G$1" pin="PA18/I2/SERCOM1+3.2"/>
-</segment>
-<segment>
-<wire x1="218.44" y1="-226.06" x2="210.82" y2="-226.06" width="0.1524" layer="91"/>
-<label x="210.82" y="-226.06" size="1.27" layer="95" font="vector" rot="R180" xref="yes"/>
-<pinref part="JP2" gate="A" pin="7"/>
 </segment>
 </net>
@@
 </segment>
 </net>
-<net name="/SS" class="0">
-<segment>
-<wire x1="320.04" y1="-83.82" x2="309.88" y2="-83.82" width="0.1524" layer="91"/>
-<label x="309.88" y="-83.82" size="1.27" layer="95" font="vector" rot="R180" xref="yes"/>
-<pinref part="U3" gate="G$1" pin="PA19/I3/SERCOM1+3.3/I2SD0"/>
-</segment>
-<segment>
-<wire x1="218.44" y1="-228.6" x2="210.82" y2="-228.6" width="0.1524" layer="91"/>
-<label x="210.82" y="-228.6" size="1.27" layer="95" font="vector" rot="R180" xref="yes"/>
-<pinref part="JP2" gate="A" pin="9"/>
-</segment>
-</net>
 <net name="SD_MOSI" class="0">
 <segment>
@@
 </segment>
 <segment>
-<wire x1="403.86" y1="-68.58" x2="419.1" y2="-68.58" width="0.1524" layer="91"/>
-<label x="419.1" y="-68.58" size="1.27" layer="95" font="vector" xref="yes"/>
-<pinref part="U3" gate="G$1" pin="PB09/I9/AIN3/SERCOM4.1"/>
-</segment>
-</net>
-<net name="FAN0_SPEED" class="0">
-<segment>
 <label x="309.88" y="-50.8" size="1.27" layer="95" font="vector" rot="R180" xref="yes"/>
 <wire x1="320.04" y1="-50.8" x2="309.88" y2="-50.8" width="0.1524" layer="91"/>
 <pinref part="U3" gate="G$1" pin="PA06/EINT6/AIN6/SERCOM0.2"/>
 </segment>
+</net>
+<net name="FAN0_SPEED" class="0">
 <segment>
 <label x="386.08" y="-162.56" size="1.27" layer="95" font="vector" rot="R180" xref="yes"/>
@@
 <junction x="396.24" y="-162.56"/>
 <pinref part="FAN1" gate="G$1" pin="3"/>
+</segment>
+<segment>
+<wire x1="403.86" y1="-68.58" x2="419.1" y2="-68.58" width="0.1524" layer="91"/>
+<label x="419.1" y="-68.58" size="1.27" layer="95" font="vector" xref="yes"/>
+<pinref part="U3" gate="G$1" pin="PB09/I9/AIN3/SERCOM4.1"/>
 </segment>
 </net>
@@
 </segment>
 </net>
+<net name="MOSI" class="0">
+<segment>
+<wire x1="320.04" y1="-83.82" x2="309.88" y2="-83.82" width="0.1524" layer="91"/>
+<label x="309.88" y="-83.82" size="1.27" layer="95" font="vector" rot="R180" xref="yes"/>
+<pinref part="U3" gate="G$1" pin="PA19/I3/SERCOM1+3.3/I2SD0"/>
+</segment>
+<segment>
+<wire x1="218.44" y1="-228.6" x2="210.82" y2="-228.6" width="0.1524" layer="91"/>
+<label x="210.82" y="-228.6" size="1.27" layer="95" font="vector" rot="R180" xref="yes"/>
+<pinref part="JP2" gate="A" pin="9"/>
+</segment>
+</net>
+<net name="/SS" class="0">
+<segment>
+<wire x1="320.04" y1="-81.28" x2="309.88" y2="-81.28" width="0.1524" layer="91"/>
+<label x="309.88" y="-81.28" size="1.27" layer="95" font="vector" rot="R180" xref="yes"/>
+<pinref part="U3" gate="G$1" pin="PA18/I2/SERCOM1+3.2"/>
+</segment>
+<segment>
+<wire x1="218.44" y1="-226.06" x2="210.82" y2="-226.06" width="0.1524" layer="91"/>
+<label x="210.82" y="-226.06" size="1.27" layer="95" font="vector" rot="R180" xref="yes"/>
+<pinref part="JP2" gate="A" pin="7"/>
+</segment>
+</net>
